File: display_v2/ph_portable_refrigerator_display_hw_v2.kicad_sch (KiCad schematic)
At the start: 39 parts, among them J1 Conn_01x01, J2 Conn_01x01, J2 Conn_01x06_Pin, J3 Conn_01x01, J4 Conn_01x01, J5 Conn_01x01, J6 LCD12PIN, J7 SIM7100-6-1-15-00-A_REVC, J9 Conn_02x08_Odd_Even, Q1 C1815_SOT23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

Commit message: Han Board MCU va board Display
Changed lines of the file:
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@@
   (symbol (lib_id "ph_lib:R0805") (at 129.413 96.012 90) (unit 1)
     (in_bom yes) (on_board yes) (dnp no)
-    (property "Reference" "R6" (at 125.603 94.742 90)
+    (property "Reference" "R6" (at 124.714 94.742 90)
       (effects (font (size 1.27 1.27)))
     )
@@
   (symbol (lib_id "ph_lib:R0805") (at 119.253 121.412 90) (unit 1)
     (in_bom yes) (on_board yes) (dnp no)
-    (property "Reference" "R3" (at 115.443 120.142 90)
+    (property "Reference" "R3" (at 114.554 120.269 90)
       (effects (font (size 1.27 1.27)))
     )
@@
   (symbol (lib_id "ph_lib:R0805") (at 119.253 116.332 90) (unit 1)
     (in_bom yes) (on_board yes) (dnp no)
-    (property "Reference" "R1" (at 115.443 115.062 90)
+    (property "Reference" "R1" (at 114.554 115.189 90)
       (effects (font (size 1.27 1.27)))
     )
@@
   (symbol (lib_id "ph_lib:R0805") (at 129.413 106.172 90) (unit 1)
     (in_bom yes) (on_board yes) (dnp no)
-    (property "Reference" "R10" (at 125.603 104.902 90)
+    (property "Reference" "R10" (at 124.714 104.902 90)
       (effects (font (size 1.27 1.27)))
     )
@@
   (symbol (lib_id "ph_lib:R0805") (at 119.253 123.952 90) (unit 1)
     (in_bom yes) (on_board yes) (dnp no)
-    (property "Reference" "R4" (at 115.443 122.682 90)
+    (property "Reference" "R4" (at 114.554 122.809 90)
       (effects (font (size 1.27 1.27)))
     )
@@
   (symbol (lib_id "ph_lib:R0805") (at 129.413 101.092 90) (unit 1)
     (in_bom yes) (on_board yes) (dnp no)
-    (property "Reference" "R8" (at 125.603 99.822 90)
+    (property "Reference" "R8" (at 124.714 99.822 90)
       (effects (font (size 1.27 1.27)))
     )
@@
   (symbol (lib_id "ph_lib:R0805") (at 129.413 103.632 90) (unit 1)
     (in_bom yes) (on_board yes) (dnp no)
-    (property "Reference" "R9" (at 125.603 102.362 90)
+    (property "Reference" "R9" (at 124.714 102.362 90)
       (effects (font (size 1.27 1.27)))
     )
@@
   (symbol (lib_id "ph_lib:R0805") (at 119.253 126.492 90) (unit 1)
     (in_bom yes) (on_board yes) (dnp no)
-    (property "Reference" "R5" (at 115.443 125.222 90)
+    (property "Reference" "R5" (at 114.554 125.349 90)
       (effects (font (size 1.27 1.27)))
     )
@@
   (symbol (lib_id "ph_lib:R0805") (at 119.253 118.872 90) (unit 1)
     (in_bom yes) (on_board yes) (dnp no)
-    (property "Reference" "R2" (at 115.443 117.602 90)
+    (property "Reference" "R2" (at 114.554 117.729 90)
       (effects (font (size 1.27 1.27)))
     )
@@
   (symbol (lib_id "ph_lib:R0805") (at 129.413 98.552 90) (unit 1)
     (in_bom yes) (on_board yes) (dnp no)
-    (property "Reference" "R7" (at 125.603 97.282 90)
-      (effects (font (size 1.27 1.27)))
-    )
+    (property "Reference" "R7" (at 124.714 97.282 90)
+      (effects (font (size 1.27 1.27)))
+    )
