File: display_v2/ph_portable_refrigerator_display_hw_v2.kicad_pcb (KiCad board)
At the start: 2 copper layers, 45 x 161.8 mm, 43 parts, among them J1 Conn_01x01, J2 Conn_01x01, J3 Conn_01x01, J4 Conn_01x01, J5 Conn_01x01, J6 LCD12PIN, J9 Conn_02x08_Odd_Even, Q1 C1815_SOT23, U1 CY8CMBR3116

Commit message: Oder PCB, Viet tai lieu mo ta hardware
Parts:
- added C1: 100nF, Capacitor_SMD:C_0805_2012Metric, F.Cu at (38.5, 187.8)
- added J1: SIM7100-6-1-15-00-A_REVC, Lib_Hien:microSIM_Card, F.Cu at (57.5, 192.9)
- added J2: Conn_01x06_Pin, Connector_PinHeader_1.27mm:PinHeader_1x06_P1.27mm_Horizontal, F.Cu at (39.5, 194.0)
Routing:
- net (no net): track 0.00 -> 102.4 mm
- net GND: vias 11 -> 51
Other:
- board size 45 x 161.8 mm -> 45 x 177.8 mm
- board text added: "3V3"
- board text added: "CLK"
- board text added: "Connect board MCU"
- board text added: "DATA"
- board text added: "DET"
- board text added: "GND"
- board text added: "IQR"
- board text added: "LCD_BL"
- board text added: "LCD_CS"
- board text added: "LCD_DC"
- board text added: "LCD_RST"
- board text added: "MOSI"
- board text added: "RST"
- board text added: "SCL"
- board text added: "SDA"
- board text added: "SPI_CLK"
- board text added: "Version: 2 Maker: P.D.H Date: 05_2023"
- board text added: "nano SIM"
- board text added: "vsim"

Commit message: update
Parts:
- removed ?: LOGO, 01phkicad:logo
