File: power_v2/GSM_Block.kicad_sch (KiCad schematic)
At the start: 41 parts, among them J1 SIM7100-6-1-15-00-A_REVC, J2 Conn_01x06_Pin, Q2 C1815_SOT23, U10 SIM_COM_A7670, U5 MIC29302WU

Commit message: Han Board MCU va board Display
Parts:
- R23: value 5.1k/1% -> 240R/1%
- R24: value 10.5k/1% -> 120R/1%
- R37: value 4.7K -> 47K
Changed lines of the file:
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@@
       (effects (font (size 1.27 1.27)) (justify left))
     )
-    (property "Value" "4.7K" (at 246.126 138.811 90)
+    (property "Value" "47K" (at 246.126 138.811 90)
       (effects (font (size 1.27 1.27)) (justify left))
     )
@@
   (symbol (lib_id "ph_lib:R0805") (at 65.532 46.736 0) (unit 1)
     (in_bom yes) (on_board yes) (dnp no) (fields_autoplaced)
-    (property "Reference" "R24" (at 67.437 45.4659 0)
-      (effects (font (size 1.27 1.27)) (justify left))
-    )
-    (property "Value" "10.5k/1%" (at 67.437 48.0059 0)
+    (property "Reference" "R24" (at 67.31 46.101 0)
+      (effects (font (size 1.27 1.27)) (justify left))
+    )
+    (property "Value" "120R/1%" (at 67.31 48.641 0)
       (effects (font (size 1.27 1.27)) (justify left))
     )
@@
   (symbol (lib_id "ph_lib:R0805") (at 65.532 39.116 0) (unit 1)
     (in_bom yes) (on_board yes) (dnp no) (fields_autoplaced)
-    (property "Reference" "R23" (at 68.072 37.8459 0)
-      (effects (font (size 1.27 1.27)) (justify left))
-    )
-    (property "Value" "5.1k/1%" (at 68.072 40.3859 0)
+    (property "Reference" "R23" (at 67.31 38.481 0)
+      (effects (font (size 1.27 1.27)) (justify left))
+    )
+    (property "Value" "240R/1%" (at 67.31 41.021 0)
       (effects (font (size 1.27 1.27)) (justify left))
     )
@@
       (effects (font (size 1.27 1.27)) (justify left))
     )
-    (property "Value" "4.7K" (at 238.506 92.075 90)
-      (effects (font (size 1.27 1.27)) (justify left))
-    )
+    (property "Value" "47K" (at 238.506 92.075 90)
+      (effects (font (size 1.27 1.27)) (justify left))
+    )

Commit message: Modify tx/rx UART0, LED GPS, pin rst/clk sim card
Parts:
- removed C1: 100nF, Capacitor_SMD:C_0805_2012Metric, symbol ph_lib:C0805
- removed J1: SIM7100-6-1-15-00-A_REVC, Lib_Hien:microSIM_Card, symbol simcard:SIM7100-6-1-15-00-A_REVC
Connections:
- net sim_clk#: now also J2.3 (Pin_3); no longer J2.5 (Pin_5)
- net sim_rst#: now also J2.5 (Pin_5); no longer J2.3 (Pin_3)
- no-connect marks 28 -> 27
Other:
- moved on the sheet: J2
